Commit message: Add test_launch.py for ROS2 testing

File: install/robot_description/share/robot_description/urdf/camera.xacro (robot description, xacro)
@@ -1,53 +1 @@
-<?xml version="1.0"?>
-<robot xmlns:xacro="http://www.ros.org/wiki/xacro">
-    <link name="camera_link">
-        <visual>
-            <geometry>
-                <mesh filename="package://robot_description/meshes/camera.dae" scale="${scale}"/>
-            </geometry>
-            <origin xyz="${-scale_num * 0.012} 0.0 ${-scale_num * 0.0116}" rpy="0.0 0.0 ${pi/2}"/>
-            <material name="black"/>
-        </visual>
-        <xacro:camera_inertia xyz="0.0 0.0 0.0" rpy="0.0 0.0 0.0"/>
-        <collision>
-            <geometry>
-                <mesh filename="package://robot_description/meshes/camera.dae" scale="${scale}"/>
-            </geometry>
-            <origin xyz="${-scale_num * 0.012} 0.0 ${-scale_num * 0.0116}" rpy="0.0 0.0 ${pi/2}"/>
-        </collision>
-    </link>
-    <joint name="base_camera_joint" type="fixed">
-        <parent link="base_link"/>
-        <child link="camera_link"/>
-        <origin xyz="${scale_num * 0.087} 0.0 ${scale_num * 0.0606}" rpy="0.0 0.0 0.0"/>
-    </joint>
-    <link name="camera_link_optical">
-    </link>
-    <joint name="camera_optical_joint" type="fixed">
-        <origin xyz="0 0 0" rpy="${-pi/2} 0 ${-pi/2}"/>
-        <parent link="camera_link"/>
-        <child link="camera_link_optical"/>
-    </joint>
-    <gazebo reference="camera_link">
-        <material>Gazebo/Gray</material>
-        <sensor name="camera_sensor" type="camera">
-            <pose>0 0 0 0 0 0</pose>
-            <visualize>true</visualize>
-            <update_rate>10.0</update_rate>
-            <camera>
-                <horizontal_fov>${60*pi/180}</horizontal_fov>
-                <image>
-                    <width>640</width>
-                    <height>480</height>
-                </image>
-                <clip>
-                    <near>0.1</near>
-                    <far>300</far>
-                </clip>
-            </camera>
-            <plugin name="camera_controller" filename="libgazebo_ros_camera.so">
-                <frame_name>camera_link_optical</frame_name>
-            </plugin>
-        </sensor>
-    </gazebo>
-</robot>
+/home/ghayth/Home_robot-master/HomeBot-ROS2-Navigation-main/src/robot_description/urdf/camera.xacro

File: install/robot_description/share/robot_description/urdf/common_properties.xacro (robot description, xacro)
@@ -1,64 +1 @@
-<?xml version="1.0"?>
-<robot xmlns:xacro="http://www.ros.org/wiki/xacro">
-    <xacro:property name="kgmm2_to_kgm2" value="1e-6" />
-    <material name="red">
-        <color rgba="0.65 0.0 0.0 1.0" />
-    </material>
-    <material name="blue">
-        <color rgba="0.0 0.0 0.65 1.0" />
-    </material>
-    <material name="black">
-        <color rgba ="0.1 0.1 0.1 1.0" />
-    </material>
-    <material name="silver">
-        <color rgba="0.75 0.75 0.75 1.0" />
-    </material>
-    <material name="gray">
-        <color rgba="0.5 0.5 0.5 1.0" />
-    </material>
-    <xacro:macro name="base_inertia" params="xyz rpy">
-        <inertial>
-            <origin xyz="${xyz}" rpy="${rpy}" />
-            <mass value="0.324" />
-            <inertia ixx="${kgmm2_to_kgm2*1321.81}" ixy="${kgmm2_to_kgm2*(-1.06e-4)}"
-                    ixz="0" iyy="${kgmm2_to_kgm2*963.45}"
-                    iyz="0" izz="${kgmm2_to_kgm2*1640.97}" />
-        </inertial>
-    </xacro:macro>
-    <xacro:macro name="motor_inertia" params="xyz rpy">
-        <inertial>
-            <origin xyz="${xyz}" rpy="${rpy}" />
-            <mass value="0.016" />
-            <inertia ixx="${kgmm2_to_kgm2*0.67}" ixy="${kgmm2_to_kgm2*(-1.41e-7)}"
-                    ixz="${kgmm2_to_kgm2*(-0.022)}" iyy="${kgmm2_to_kgm2*1.43}"
-                    iyz="${kgmm2_to_kgm2*(-1.12e-4)}" izz="${kgmm2_to_kgm2*1.651}" />
-        </inertial>
-    </xacro:macro>
-    <xacro:macro name="wheel_inertia" params="xyz rpy">
-        <inertial>
-            <origin xyz="${xyz}" rpy="${rpy}" />
-            <mass value="0.023" />
-            <inertia ixx="${kgmm2_to_kgm2*19.31}" ixy="${kgmm2_to_kgm2*(-2.91e-8)}"
-                    ixz="${kgmm2_to_kgm2*(-4.18e-8)}" iyy="${kgmm2_to_kgm2*9.80}"
-                    iyz="${kgmm2_to_kgm2*(4.49e-7)}" izz="${kgmm2_to_kgm2*9.81}" />
-        </inertial>
-    </xacro:macro>
-    <xacro:macro name="camera_inertia" params="xyz rpy">
-        <inertial>
-            <origin xyz="${xyz}" rpy="${rpy}" />
-            <mass value="0.04" />
-            <inertia ixx="${kgmm2_to_kgm2*3.04}" ixy="${kgmm2_to_kgm2*0.004}"
-                    ixz="${kgmm2_to_kgm2*(1.31e-4)}" iyy="${kgmm2_to_kgm2*32.45}"
-                    iyz="${kgmm2_to_kgm2*(-0.017)}" izz="${kgmm2_to_kgm2*32.46}" />
-        </inertial>
-    </xacro:macro>
-    <xacro:macro name="lidar_inertia" params="xyz rpy">
-        <inertial>
-            <origin xyz="${xyz}" rpy="${rpy}" />
-            <mass value="0.152" />
-            <inertia ixx="${kgmm2_to_kgm2*98.88}" ixy="${kgmm2_to_kgm2*0.453}"
-                    ixz="${kgmm2_to_kgm2*(-0.779)}" iyy="${kgmm2_to_kgm2*62.04}"
-                    iyz="${kgmm2_to_kgm2*(-13.95)}" izz="${kgmm2_to_kgm2*123.1}" />
-        </inertial>
-    </xacro:macro>
-</robot>
+/home/ghayth/Home_robot-master/HomeBot-ROS2-Navigation-main/src/robot_description/urdf/common_properties.xacro

File: install/robot_description/share/robot_description/urdf/lidar.xacro (robot description, xacro)
@@ -1,57 +1 @@
-<?xml version="1.0"?>
-<robot xmlns:xacro="http://www.ros.org/wiki/xacro">
-    <link name="lidar_link">
-        <visual>
-            <geometry>
-                <mesh filename="package://robot_description/meshes/rplidar.dae" scale="${scale}"/>
-            </geometry>
-            <origin xyz="0.0 0.0 0.0" rpy="0.0 0.0 ${pi}"/>
-            <material name="black"/>
-        </visual>
-        <xacro:lidar_inertia xyz="0.0 0.0 0.0" rpy="0.0 0.0 0.0"/>
-        <collision>
-            <geometry>
-                <mesh filename="package://robot_description/meshes/rplidar.dae" scale="${scale}"/>
-            </geometry>
-            <origin xyz="0.0 0.0 0.0" rpy="0.0 0.0 0.0"/>
-        </collision>
-    </link>
-    <joint name="base_lidar_joint" type="fixed">
-        <parent link="base_link"/>
-        <child link="lidar_link"/>
-        <origin xyz="0.0 0.0 ${scale_num * 0.1116}" rpy="0.0 0.0 ${-pi/2}"/>
-    </joint>
-    <link name="laser_frame" />
-    <joint name="lidar_laser_joint" type="fixed">
-        <parent link="lidar_link"/>
-        <child link="laser_frame"/>
-        <origin xyz="0.0 0.0 ${scale_num * 0.025101}" rpy="0.0 0.0 0.0"/>
-    </joint>
-    <gazebo reference="laser_frame">
-        <sensor name="laser" type="ray">
-            <pose> 0 0 0 0 0 0 </pose>
-            <visualize>true</visualize>
-            <update_rate>10</update_rate>
-            <ray>
-                <scan>
-                    <horizontal>
-                        <samples>720</samples>
-                        <min_angle>-3.14</min_angle>
-                        <max_angle>3.14</max_angle>
-                    </horizontal>
-                </scan>
-                <range>
-                    <min>0.1</min>
-                    <max>12</max>
-                </range>
-            </ray>
-            <plugin name="laser_controller" filename="libgazebo_ros_ray_sensor.so">
-                <ros>
-                    <argument>~/out:=scan</argument>
-                </ros>
-                <output_type>sensor_msgs/LaserScan</output_type>
-                <frame_name>laser_frame</frame_name>
-            </plugin>
-        </sensor>
-    </gazebo>
-</robot>
+/home/ghayth/Home_robot-master/HomeBot-ROS2-Navigation-main/src/robot_description/urdf/lidar.xacro

File: install/robot_description/share/robot_description/urdf/mobile_robot.urdf.xacro (robot description, xacro)
@@ -1,8 +1 @@
-<?xml version="1.0"?>
-<robot name="my_robot" xmlns:xacro="http://www.ros.org/wiki/xacro">
-    <xacro:include filename="common_properties.xacro" />
-    <xacro:include filename="mobile_robot_base.xacro" />
-    <xacro:include filename="mobile_robot_gazebo.xacro" />
-    <xacro:include filename="lidar.xacro" />
-    <xacro:include filename="camera.xacro" />
-</robot>
+/home/ghayth/Home_robot-master/HomeBot-ROS2-Navigation-main/src/robot_description/urdf/mobile_robot.urdf.xacro

File: install/robot_description/share/robot_description/urdf/mobile_robot_base.xacro (robot description, xacro)
@@ -1,98 +1 @@
-<?xml version="1.0"?>
-<robot xmlns:xacro="http://www.ros.org/wiki/xacro">
-    <!-- The 'scale_num' and 'scale' properties are used to adjust the size of the robot's visual and collision meshes within the simulation environment.
-     This is particularly useful for visualizing the transform frames (TFs) more clearly during development and debugging.
-     The default scale is set to 1.0, which represents the actual size of the robot. It can be adjusted as necessary for better visibility. -->
-    <xacro:property name="scale_num" value="1.0" />
-    <xacro:property name="scale" value="${scale_num} ${scale_num} ${scale_num}" />
-    <link name="base_footprint" />
-    <link name="base_link">
-        <visual>
-            <geometry>
-                <mesh filename="package://robot_description/meshes/base_link.dae"
-                    scale="${scale}"/>
-            </geometry>
-            <origin xyz="0.0 0.0 0.0" rpy="0.0 0.0 ${-pi/2}"/>
-            <material name="black"/>
-        </visual>
-        <xacro:base_inertia xyz="0.0 0.0 0.0" rpy="0.0 0.0 0.0"/>
-        <collision>
-            <geometry>
-                <mesh filename="package://robot_description/meshes/base_link.dae"
-                    scale="${scale}"/>
-            </geometry>
-            <origin xyz="0.0 0.0 0.0" rpy="0.0 0.0 ${-pi/2}"/>
-        </collision>
-    </link>
-    <joint name="base_joint" type="fixed">
-        <parent link="base_footprint"/>
-        <child link="base_link"/>
-        <origin xyz="0.0 0.0 ${scale_num * 0.028}" rpy="0.0 0.0 0.0"/>
-    </joint>
-    <xacro:macro name="motor_link" params="prefix">
-        <link name="${prefix}_motor_link">
-            <visual>
-                <geometry>
-                    <mesh filename="package://robot_description/meshes/motor.dae"
-                        scale="${scale}"/>
-                </geometry>
-                <origin xyz="0.0 0.0 0.0" rpy="0.0 0.0 0.0"/>
-                <material name="silver"/>
-            </visual>
-            <xacro:motor_inertia xyz="0.0 0.0 0.0" rpy="0.0 0.0 0.0"/>
-            <collision>
-                <geometry>
-                    <mesh filename="package://robot_description/meshes/motor.dae"
-                        scale="${scale}"/>
-                </geometry>
-                <origin xyz="0.0 0.0 0.0" rpy=" 0.0  0.0 0.0"/>
-            </collision>
-        </link>
-    </xacro:macro>
-    <xacro:motor_link prefix="left" />
-    <xacro:motor_link prefix="right" />
-    <joint name="base_right_motor_joint" type="fixed">
-        <parent link="base_link"/>
-        <child link="right_motor_link"/>
-        <origin xyz=" 0.0 ${-scale_num * 0.03348} ${scale_num*0.008}" rpy="0.0 0.0 ${-pi/2}"/>
-    </joint>
-        <joint name="base_left_motor_joint" type="fixed">
-        <parent link="base_link"/>
-        <child link="left_motor_link"/>
-        <origin xyz=" 0.0 ${scale_num * 0.03348} ${scale_num*0.008}" rpy=" 0.0  0.0 ${pi/2}"/>
-    </joint>
-    <xacro:macro name="wheel_link" params="prefix rotation">
-        <link name="${prefix}_wheel_link">
-            <visual>
-                <geometry>
-                    <mesh filename="package://robot_description/meshes/wheel.dae"
-                        scale="${scale}"/>
-                </geometry>
-                <origin xyz="0.0 0.0 0.0" rpy=" 0.0  0.0 ${rotation}"/>
-                <material name="gray"/>
-            </visual>
-            <xacro:motor_inertia xyz="0.0 0.0 0.0" rpy="0.0 0.0 0.0"/>
-            <collision>
-                <geometry>
-                    <mesh filename="package://robot_description/meshes/wheel.dae"
-                        scale="${scale}"/>
-                </geometry>
-                <origin xyz="0.0 0.0 0.0" rpy="0 0.0 ${rotation}"/>
-            </collision>
-        </link>
-    </xacro:macro>
-    <xacro:wheel_link prefix="right" rotation="${pi/2}"/>
-    <xacro:wheel_link prefix="left" rotation="${-pi/2}"/>
-    <joint name="left_motor_wheel_joint" type="continuous">
-        <parent link="left_motor_link"/>
-        <child link="left_wheel_link"/>
-        <origin xyz="${scale_num * 0.01992} 0.0 0.0" rpy="0.0 0.0 ${pi/2}"/>
-        <axis xyz=" 0.0 -1 0.0"/>
-    </joint>
-    <joint name="right_motor_wheel_joint" type="continuous">
-        <parent link="right_motor_link"/>
-        <child link="right_wheel_link"/>
-        <origin xyz="${scale_num * 0.01992} 0.0 0.0" rpy="0 0 ${-pi/2}"/>
-        <axis xyz="0.0 -1.0 0.0"/>
-    </joint>
-</robot>
+/home/ghayth/Home_robot-master/HomeBot-ROS2-Navigation-main/src/robot_description/urdf/mobile_robot_base.xacro

File: install/robot_description/share/robot_description/urdf/mobile_robot_gazebo.xacro (robot description, xacro)
@@ -1,43 +1 @@
-<?xml version="1.0"?>
-<robot xmlns:xacro="http://www.ros.org/wiki/xacro">
-    <gazebo reference="base_link">
-        <material>Gazebo/Black</material>
-        <mu1 value="0.01"/>
-        <mu2 value="0.01"/>
-    </gazebo>
-    <gazebo reference="left_motor_link">
-        <material>Gazebo/Red</material>
-    </gazebo>
-    <gazebo reference="right_motor_link">
-        <material>Gazebo/Red</material>
-    </gazebo>
-    <gazebo reference="left_wheel_link">
-        <material>Gazebo/Grey</material>
-        <mu1 value="0.1"/>
-        <mu2 value="0.1"/>
-    </gazebo>
-    <gazebo reference="right_wheel_link">
-        <mu1 value="0.1"/>
-        <mu2 value="0.1"/>
-        <material>Gazebo/Grey</material>
-    </gazebo>
-    <gazebo>
-        <plugin name="diff_drive_controller" filename="libgazebo_ros_diff_drive.so">
-            <!-- wheels -->
-            <left_joint>left_motor_wheel_joint</left_joint>
-            <right_joint>right_motor_wheel_joint</right_joint>
-            <!-- kinematics -->
-            <wheel_separation>${scale_num*0.057504}</wheel_separation>
-            <wheel_diameter>${0.072*scale_num}</wheel_diameter>
-            <!-- limits -->
-            <max_wheel_torque>20</max_wheel_torque>
-            <max_wheel_acceleration>1.0</max_wheel_acceleration>
-            <!-- output -->
-            <odometry_frame>odom</odometry_frame>
-            <robot_base_frame>base_footprint</robot_base_frame>
-            <publish_odom>true</publish_odom>
-            <publish_odom_tf>true</publish_odom_tf>
-            <publish_wheel_tf>true</publish_wheel_tf>
-        </plugin>
-    </gazebo>
-</robot>
+/home/ghayth/Home_robot-master/HomeBot-ROS2-Navigation-main/src/robot_description/urdf/mobile_robot_gazebo.xacro
